File: hardware/node-prototype/microphone.kicad_sch (KiCad schematic)
At the start: 14 parts, among them Q3 2N7002, U10 MAX9814

Commit message: Double check schematic
Parts:
- added C46: 1nF, Capacitor_SMD:C_0603_1608Metric_Pad1.08x0.95mm_HandSolder, symbol Device:C
- added C47: 100nF, Capacitor_SMD:C_0603_1608Metric, symbol Device:C
- added R49: 130R, Resistor_SMD:R_0603_1608Metric, symbol Device:R
- added TP2 (x3): TestPoint, TestPoint:TestPoint_Pad_D2.0mm, symbol Connector:TestPoint
- C31, C33, C34, C35: symbol Device:C_Polarized -> Device:C
- C32: footprint Capacitor_SMD:C_0603_1608Metric -> Capacitor_SMD:C_0603_1608Metric_Pad1.08x0.95mm_HandSolder; symbol Device:C_Polarized -> Device:C
- MK1: value Microphone_Condenser -> CMA-4544PF-W
- R36: value 68R -> 270R
Connections:
- net GND: now also MK1.2 (+), C46.2, C47.2; no longer MK1.1 (-), R29.2
- net VDDA: now also C47.1
- net at C31.2: now also MK1.1 (-), R29.2, TP2.1; no longer MK1.2 (+)
- net MIC_AUDIO: no longer names the net of U10.6 (MICOUT)
- net MIC_AUDIO: now also R49.1, TP2.1
- net MIC_A/R renamed A/R
- net MIC_GAIN renamed GAIN
- net ~{MIC_SHDN} renamed ~{SHDN}
- net ~{SHDN}: now also TP2.1
- new net AUDIO: C46.1, R49.2
Other:
- note added: "Anti Aliasing Low-Pass fc=1.2MHz"
- moved on the sheet: D4, MK1, R29, R30, R31, R36

Commit message: prepare for production
Parts:
- MK1: now not fitted
- TP2: now left out of the parts list
Changed lines of the file:
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@@
   )
   (symbol (lib_id "Connector:TestPoint") (at 162.56 71.755 0) (unit 1)
-    (in_bom yes) (on_board yes) (dnp no) (fields_autoplaced)
+    (in_bom no) (on_board yes) (dnp no) (fields_autoplaced)
     (property "Reference" "TP2" (at 165.1 67.183 0)
       (effects (font (size 1.27 1.27)) (justify left))
@@
   )
   (symbol (lib_id "Connector:TestPoint") (at 71.755 128.27 0) (unit 1)
-    (in_bom yes) (on_board yes) (dnp no) (fields_autoplaced)
+    (in_bom no) (on_board yes) (dnp no) (fields_autoplaced)
     (property "Reference" "TP2" (at 74.295 123.698 0)
       (effects (font (size 1.27 1.27)) (justify left))
@@
   )
   (symbol (lib_id "Device:Microphone_Condenser") (at 68.58 135.89 0) (mirror x) (unit 1)
-    (in_bom yes) (on_board yes) (dnp no)
+    (in_bom yes) (on_board yes) (dnp yes)
     (property "Reference" "MK1" (at 62.23 135.89 90)
       (effects (font (size 1.27 1.27)))
@@
   )
   (symbol (lib_id "Connector:TestPoint") (at 201.93 99.06 0) (unit 1)
-    (in_bom yes) (on_board yes) (dnp no) (fields_autoplaced)
+    (in_bom no) (on_board yes) (dnp no) (fields_autoplaced)
     (property "Reference" "TP2" (at 204.47 94.488 0)
       (effects (font (size 1.27 1.27)) (justify left))
